Commit message: added ros2 control and mecanum drive controller

File: description/gazebo_control.xacro (robot description, xacro)
@@ -2,10 +2,15 @@
 <robot xmlns:xacro="http://www.ros.org/wiki/xacro"  name="robot">
     <gazebo>
-        <plugin name="diff_drive" filename="libgazebo_ros_diff_drive.so">
+        <plugin name="diff_drive_controller" filename="libgazebo_ros_diff_drive.so">
             <!-- WHEEL INFORMATION-->
-            <left_joint>left_wheel_joint</left_joint>
-            <right_joint>right_wheel_joint</right_joint>
-            <wheel_separation>0.35</wheel_separation>
-            <wheel_diameter>0.1</wheel_diameter>
+            <num_wheel_pairs>2</num_wheel_pairs>
+            <left_joint>front_left_wheel_joint</left_joint>
+            <left_joint>back_left_wheel_joint</left_joint>
+            <right_joint>front_right_wheel_joint</right_joint>
+            <right_joint>back_right_wheel_joint</right_joint>
+            <wheel_separation>0.17</wheel_separation>
+            <wheel_separation>0.17</wheel_separation>
+            <wheel_diameter>0.06</wheel_diameter>
+            <wheel_diameter>0.06</wheel_diameter>
             <!-- Limits -->
             <max_wheel_torque>200</max_wheel_torque>

File: description/robot.urdf.xacro (robot description, xacro)
@@ -2,4 +2,4 @@
 <robot xmlns:xacro="http://www.ros.org/wiki/xacro"  name="robot">
  <xacro:include filename="robot_core.xacro"/>
-<xacro:include filename="gazebo_control.xacro"/>
+ <xacro:include filename="ros2_control.xacro"/>
 </robot>

File: description/robot_core.xacro (robot description, xacro)
@@ -20,19 +20,19 @@
         <parent link="base_link"/>
         <child link="chassis"/>
-        <origin xyz="-0.1 0.0 0.0"/>
+        <origin xyz="-0.11 0.0 0.0"/>
     </joint>
     <!-- CHASSIS LINK-->
     <link name="chassis">
         <visual>
-            <origin xyz="0.15 0 0.075"/>
+            <origin xyz="0.11 0 0.090"/>
             <geometry>
-                <box size="0.3 0.3 0.15"/>
+                <box size="0.22 0.17 0.11"/>
             </geometry>
             <material name="white"/>
         </visual>
         <collision>
-            <origin xyz="0.15 0 0.075"/>
+            <origin xyz="0.15 0 0.090"/>
             <geometry>
-                <box size="0.3 0.3 0.15"/>
+                <box size="0.22 0.17 0.15"/>
             </geometry>
         </collision>
@@ -45,14 +45,15 @@
     </gazebo>
     <!-- LEFT WHEEL LINK-->
-    <joint name="left_wheel_joint" type="continuous">
+                <!-- FRONT -->
+    <joint name="front_left_wheel_joint" type="continuous">
         <parent link="base_link"/>
-        <child link="left_wheel"/>
-        <origin xyz="0 0.175 0" rpy="-${pi/2} 0 0"/>
+        <child link="front_left_wheel"/>
+        <origin xyz="0.085 0.1 0" rpy="-${pi/2} 0 0"/>
         <axis xyz="0.0 0.0 1.0"/>
     </joint>
-    <link name="left_wheel">
+    <link name="front_left_wheel">
     <visual>
         <geometry>
-            <cylinder radius="0.05" length="0.04"/>
+            <cylinder radius="0.03" length="0.02"/>
         </geometry>
         <material name="blue"/>
@@ -60,25 +61,25 @@
     <collision>
         <geometry>
-            <cylinder radius="0.05" length="0.04"/>
+            <cylinder radius="0.03" length="0.02"/>
         </geometry>
     </collision>
-    <xacro:inertial_cylinder mass="0.1" length="0.04" radius="0.05">
+    <xacro:inertial_cylinder mass="0.1" length="0.02" radius="0.03">
         <origin xyz="0 0 0" rpy="0 0 0"/>
     </xacro:inertial_cylinder>
     </link>
-    <gazebo reference="left_wheel">
+    <gazebo reference="front_left_wheel">
         <material>Gazebo/Blue</material>
     </gazebo>
-    <!-- RIGHT WHEEL LINK-->
-    <joint name="right_wheel_joint" type="continuous">
+                <!-- BACK -->
+    <joint name="back_left_wheel_joint" type="continuous">
         <parent link="base_link"/>
-        <child link="right_wheel"/>
-        <origin xyz="0 -0.175 0" rpy="${pi/2} 0 0"/>
-        <axis xyz="0.0 0.0 -1.0"/>
+        <child link="back_left_wheel"/>
+        <origin xyz="-0.085 0.1 0" rpy="-${pi/2} 0 0"/>
+        <axis xyz="0.0 0.0 1.0"/>
     </joint>
-    <link name="right_wheel">
+    <link name="back_left_wheel">
     <visual>
         <geometry>
-            <cylinder radius="0.05" length="0.04"/>
+            <cylinder radius="0.03" length="0.02"/>
         </geometry>
         <material name="blue"/>
@@ -86,40 +87,66 @@
     <collision>
         <geometry>
-            <cylinder radius="0.05" length="0.04"/>
+            <cylinder radius="0.03" length="0.02"/>
         </geometry>
     </collision>
-    <xacro:inertial_cylinder mass="0.1" length="0.04" radius="0.05">
+    <xacro:inertial_cylinder mass="0.1" length="0.02" radius="0.03">
         <origin xyz="0 0 0" rpy="0 0 0"/>
     </xacro:inertial_cylinder>
     </link>
-    <gazebo reference="right_wheel">
+    <gazebo reference="back_left_wheel">
         <material>Gazebo/Blue</material>
     </gazebo>
-    <!-- CASTER WHEEL LINK-->
-    <joint name="caster_wheel_joint" type="fixed">
-    <parent link="chassis"/>
-    <child link="caster_wheel"/>
-    <origin xyz="0.24 0 0" />
+    <!-- RIGHT WHEEL LINK-->
+            <!--FRONT-->
+    <joint name="front_right_wheel_joint" type="continuous">
+        <parent link="base_link"/>
+        <child link="front_right_wheel"/>
+        <origin xyz="0.085 -0.1 0" rpy="${pi/2} 0 0"/>
+        <axis xyz="0.0 0.0 -1.0"/>
     </joint>
-    <link name="caster_wheel">
+    <link name="front_right_wheel">
     <visual>
         <geometry>
-            <sphere radius="0.05"/>
+            <cylinder radius="0.03" length="0.02"/>
         </geometry>
-        <material name="black"/>
+        <material name="blue"/>
     </visual>
     <collision>
-            <geometry>
-                <sphere radius="0.05"/>
-            </geometry>
+        <geometry>
+            <cylinder radius="0.03" length="0.02"/>
+        </geometry>
     </collision>
-    <xacro:inertial_sphere mass="0.1" radius="0.05">
+    <xacro:inertial_cylinder mass="0.1" length="0.02" radius="0.03">
         <origin xyz="0 0 0" rpy="0 0 0"/>
-    </xacro:inertial_sphere>
+    </xacro:inertial_cylinder>
     </link>
-    <gazebo reference="caster_wheel">
-        <material>Gazebo/Black</material>
-        <mu1 value="0.001"/>
-        <mu2 value="0.001"/>
+    <gazebo reference="front_right_wheel">
+        <material>Gazebo/Blue</material>
+    </gazebo>
+            <!--BACK-->
+    <joint name="back_right_wheel_joint" type="continuous">
+        <parent link="base_link"/>
+        <child link="back_right_wheel"/>
+        <origin xyz="-0.085 -0.1 0" rpy="${pi/2} 0 0"/>
+        <axis xyz="0.0 0.0 -1.0"/>
+    </joint>
+    <link name="back_right_wheel">
+    <visual>
+        <geometry>
+            <cylinder radius="0.03" length="0.02"/>
+        </geometry>
+        <material name="blue"/>
+    </visual>
+    <collision>
+        <geometry>
+            <cylinder radius="0.03" length="0.02"/>
+        </geometry>
+    </collision>
+    <xacro:inertial_cylinder mass="0.1" length="0.02" radius="0.03">
+        <origin xyz="0 0 0" rpy="0 0 0"/>
+    </xacro:inertial_cylinder>
+    </link>
+    <gazebo reference="back_right_wheel">
+        <material>Gazebo/Blue</material>
     </gazebo>
 </robot>
