Commit message: edited ros2_control description to use new mecanum_drive_stm hardware interface

File: description/ros2_control.xacro (robot description, xacro)
@@ -1,4 +1,35 @@
 <?xml version="1.0"?>
 <robot xmlns:xacro="http://www.ros.org/wiki/xacro">
+    <ros2_control name="RealRobot" type="system">
+        <hardware>
+          <plugin>mecanum_drive_stm/MecanumDriveSTMHardware</plugin>
+            <param name="front_left_wheel_name">front_left_wheel_joint</param>
+            <param name="front_right_wheel_name">front_right_wheel_joint</param>
+            <param name="back_left_wheel_name">back_left_wheel_joint</param>
+            <param name="back_right_wheel_name">back_right_wheel_joint</param>
+            <param name="loop_rate">60</param>
+            <param name="device">/dev/ttyACM0</param>
+            <param name="baud_rate">9600</param>
+            <param name="timeout_ms">3000</param>
+            <param name="enc_counts_per_rev">3436</param>
+        </hardware>
+        <joint name="front_left_wheel_joint">
+            <command_interface name="velocity"/>
+            <state_interface name="velocity"/>
+        </joint>
+        <joint name="back_left_wheel_joint">
+            <command_interface name="velocity"/>
+            <state_interface name="velocity"/>
+        </joint>
+        <joint name="front_right_wheel_joint">
+            <command_interface name="velocity"/>
+            <state_interface name="velocity"/>
+        </joint>
+        <joint name="back_right_wheel_joint">
+            <command_interface name="velocity"/>
+            <state_interface name="velocity"/>
+        </joint>
+    </ros2_control>
+<!--
     <ros2_control name="GazeboSystem" type="system">
         <hardware>
@@ -38,4 +69,5 @@
         </joint>
     </ros2_control>
+-->
     <gazebo>
         <plugin name="gazebo_ros2_control" filename="libgazebo_ros2_control.so">
