Commit message: added twist_converter to convert twist messages to twistStamped, added joystick control

File: description/robot_core.xacro (robot description, xacro)
@@ -32,11 +32,11 @@
         </visual>
         <collision>
-            <origin xyz="0.15 0 0.090"/>
+            <origin xyz="0.11 0 0.090"/>
             <geometry>
-                <box size="0.22 0.17 0.15"/>
+                <box size="0.22 0.17 0.11"/>
             </geometry>
         </collision>
-        <xacro:inertial_box mass="0.5" x="0.3" y="0.5" z="0.15">
-        <origin xyz="0.15 0 0.075" rpy="0 0 0" />
+        <xacro:inertial_box mass="0.5" x="0.22" y="0.17" z="0.11">
+        <origin xyz="0.11 0 0.090" rpy="0 0 0" />
         </xacro:inertial_box>
     </link>
@@ -61,5 +61,5 @@
     <collision>
         <geometry>
-            <cylinder radius="0.03" length="0.02"/>
+            <sphere radius="0.03"/>
         </geometry>
     </collision>
@@ -87,5 +87,5 @@
     <collision>
         <geometry>
-            <cylinder radius="0.03" length="0.02"/>
+            <sphere radius="0.03"/>
         </geometry>
     </collision>
@@ -114,5 +114,5 @@
     <collision>
         <geometry>
-            <cylinder radius="0.03" length="0.02"/>
+            <sphere radius="0.03"/>
         </geometry>
     </collision>
@@ -140,5 +140,5 @@
     <collision>
         <geometry>
-            <cylinder radius="0.03" length="0.02"/>
+            <sphere radius="0.03"/>
         </geometry>
     </collision>

Commit message: edited encoder counts parameter

File: description/robot_core.xacro (robot description, xacro)
@@ -18,6 +18,5 @@
     </material>
     <!-- BASE LINK-->
-    <link name="base_link">
-    </link>
+    <link name="base_link"/>
     <joint name="chassis_joint" type="fixed">
         <parent link="base_link"/>

File: description/ros2_control.xacro (robot description, xacro)
@@ -1,5 +1,4 @@
 <?xml version="1.0"?>
 <robot xmlns:xacro="http://www.ros.org/wiki/xacro">
-<!--
     <ros2_control name="RealRobot" type="system">
         <hardware>
@@ -13,5 +12,6 @@
             <param name="baud_rate">115200</param>
             <param name="timeout_ms">3000</param>
-            <param name="enc_counts_per_rev">3436</param>
+            <param name="front_enc_counts_per_rev">30</param>
+            <param name="back_enc_counts_per_rev">718</param>
         </hardware>
         <joint name="front_left_wheel_joint">
@@ -32,5 +32,5 @@
         </joint>
     </ros2_control>
--->
+<!--
     <ros2_control name="GazeboSystem" type="system">
         <hardware>
@@ -70,4 +70,5 @@
         </joint>
     </ros2_control>
+-->
     <gazebo>
         <plugin name="gazebo_ros2_control" filename="libgazebo_ros2_control.so">

Commit message: Fixed: odom frame visibility on rviz, mecanum_cont publishing twistStamped messages, straffing

File: description/robot_core.xacro (robot description, xacro)
@@ -51,5 +51,5 @@
         <parent link="base_link"/>
         <child link="front_left_wheel"/>
-        <origin xyz="0.085 0.1 0" rpy="-${pi/2} 0 0"/>
+        <origin xyz="0.1125 0.1 0" rpy="-${pi/2} 0 0"/>
         <axis xyz="0.0 0.0 1.0"/>
     </joint>
@@ -77,5 +77,5 @@
         <parent link="base_link"/>
         <child link="back_left_wheel"/>
-        <origin xyz="-0.085 0.1 0" rpy="-${pi/2} 0 0"/>
+        <origin xyz="-0.1125 0.1 0" rpy="-${pi/2} 0 0"/>
         <axis xyz="0.0 0.0 1.0"/>
     </joint>
@@ -104,5 +104,5 @@
         <parent link="base_link"/>
         <child link="front_right_wheel"/>
-        <origin xyz="0.085 -0.1 0" rpy="${pi/2} 0 0"/>
+        <origin xyz="0.1125 -0.1 0" rpy="${pi/2} 0 0"/>
         <axis xyz="0.0 0.0 -1.0"/>
     </joint>
@@ -130,5 +130,5 @@
         <parent link="base_link"/>
         <child link="back_right_wheel"/>
-        <origin xyz="-0.085 -0.1 0" rpy="${pi/2} 0 0"/>
+        <origin xyz="-0.1125 -0.1 0" rpy="${pi/2} 0 0"/>
         <axis xyz="0.0 0.0 -1.0"/>
     </joint>

File: description/ros2_control.xacro (robot description, xacro)
@@ -1,4 +1,5 @@
 <?xml version="1.0"?>
 <robot xmlns:xacro="http://www.ros.org/wiki/xacro">
+ <!--
     <ros2_control name="RealRobot" type="system">
         <hardware>
@@ -9,5 +10,5 @@
             <param name="back_right_wheel_name">back_right_wheel_joint</param>
             <param name="loop_rate">60</param>
-            <param name="device">/dev/ttyACM0</param>
+            <param name="device">/dev/serial0</param>
             <param name="baud_rate">115200</param>
             <param name="timeout_ms">3000</param>
@@ -32,5 +33,5 @@
         </joint>
     </ros2_control>
-<!--
+-->
     <ros2_control name="GazeboSystem" type="system">
         <hardware>
@@ -70,5 +71,4 @@
         </joint>
     </ros2_control>
--->
     <gazebo>
         <plugin name="gazebo_ros2_control" filename="libgazebo_ros2_control.so">
